Commit message: fix: modify so101 joint limits for real hardware safety

File: src/humanoid/robots/assets/so101/urdf/so101.urdf (robot description, URDF)
Before this commit: robot so101_new_calib, 8 links, 7 joints
Joints:
- joint elbow_flex: limit lower=-1.69 upper=1.69 effort=10 velocity=10 -> lower=-1.55 upper=1.55 effort=10 velocity=10
- joint shoulder_lift: limit lower=-1.74533 upper=1.74533 effort=10 velocity=10 -> lower=-1.55 upper=1.55 effort=10 velocity=10
- joint shoulder_pan: limit lower=-1.91986 upper=1.91986 effort=10 velocity=10 -> lower=-1.57 upper=1.57 effort=10 velocity=10
- joint wrist_flex: limit lower=-1.65806 upper=1.65806 effort=10 velocity=10 -> lower=-1.6 upper=1.6 effort=10 velocity=10

Commit message: feat: use pink for OSC

File: src/humanoid/robots/assets/so101/urdf/so101.urdf (robot description, URDF)
Before this commit: robot so101_new_calib, 8 links, 7 joints
Joints:
- joint shoulder_pan: limit lower=-1.57 upper=1.57 effort=10 velocity=10 -> lower=-1.91986 upper=1.91986 effort=10 velocity=10
