Commit message: fix: convert .dae to .stl for pand robot viz

File: src/humanoid/robots/assets/panda/urdf/panda.urdf (robot description, URDF)
Before this commit: robot panda, 13 links, 12 joints
Links:
- link panda_hand: geometry collision mesh filename=package://panda/meshes/collision/hand.stl; visual mesh filename=package://panda/meshes/visual/hand.stl
- link panda_leftfinger: geometry collision box size=17.5e-3 15.2e-3 18.5e-3; collision box size=17.5e-3 7e-3 23.5e-3
- link panda_link0: geometry collision mesh filename=package://panda/meshes/collision/link0.stl; visual mesh filename=package://panda/meshes/visual/link0.stl
- link panda_link1: geometry collision mesh filename=package://panda/meshes/collision/link1.stl; visual mesh filename=package://panda/meshes/visual/link1.stl
- link panda_link2: geometry collision mesh filename=package://panda/meshes/collision/link2.stl; visual mesh filename=package://panda/meshes/visual/link2.stl
- link panda_link3: geometry collision mesh filename=package://panda/meshes/collision/link3.stl; visual mesh filename=package://panda/meshes/visual/link3.stl
- link panda_link4: geometry collision mesh filename=package://panda/meshes/collision/link4.stl; visual mesh filename=package://panda/meshes/visual/link4.stl
- link panda_link5: geometry collision mesh filename=package://panda/meshes/collision/link5.stl; visual mesh filename=package://panda/meshes/visual/link5.stl
- link panda_link6: geometry collision mesh filename=package://panda/meshes/collision/link6.stl; visual mesh filename=package://panda/meshes/visual/link6.stl
- link panda_link7: geometry collision mesh filename=package://panda/meshes/collision/link7.stl; visual mesh filename=package://panda/meshes/visual/link7.stl
- link panda_rightfinger: geometry collision box size=17.5e-3 15.2e-3 18.5e-3; collision box size=17.5e-3 7e-3 23.5e-3

File: src/humanoid/robots/assets/panda/urdf/panda_collision.urdf (robot description, URDF)
Before this commit: robot panda, 13 links, 12 joints
Links:
- link panda_hand: geometry collision cylinder length=0.15 radius=0.05; collision sphere radius=0.05
- link panda_leftfinger: geometry collision cylinder length=0.03 radius=0.015; collision sphere radius=0.015
- link panda_link0: geometry collision cylinder length=0.03 radius=0.09; collision sphere radius=0.09
- link panda_link1: geometry collision cylinder length=0.283 radius=0.09; collision sphere radius=0.09
- link panda_link2: geometry collision cylinder length=0.12 radius=0.09; collision sphere radius=0.09
- link panda_link3: geometry collision cylinder length=0.15 radius=0.09; collision sphere radius=0.09
- link panda_link4: geometry collision cylinder length=0.12 radius=0.09; collision sphere radius=0.09
- link panda_link5: geometry collision cylinder length=0.1 radius=0.09; collision cylinder length=0.14 radius=0.055
- link panda_link6: geometry collision cylinder length=0.08 radius=0.08; collision sphere radius=0.08
- link panda_link7: geometry collision cylinder length=0.01 radius=0.045; collision cylinder length=0.14 radius=0.07
- link panda_rightfinger: geometry collision cylinder length=0.03 radius=0.015; collision sphere radius=0.015
