Commit message: fix: use revolute w/o limits for wheels in elrobot_mobile
chore: run formatting + clean up elrobot + elrobot_mobile URDFs

File: src/humanoid/robots/assets/elrobot_mobile/urdf/elrobot_mobile.urdf (robot description, URDF)
Before this commit: robot elrobot_mobile, 31 links, 30 joints
Links:
- removed link omni_wheel_mount_v5
- removed link omni_wheel_mount_v5_1
- removed link omni_wheel_mount_v5_2
- added link omni_wheel_mount, mass 1.57415e-05; visual mesh filename=package://elrobot_mobile/meshes/omni_wheel_mount.obj scale=1 1 1
- added link omni_wheel_mount_1, mass 1.57415e-05; visual mesh filename=package://elrobot_mobile/meshes/omni_wheel_mount.obj scale=1 1 1
- added link omni_wheel_mount_2, mass 1.57415e-05; visual mesh filename=package://elrobot_mobile/meshes/omni_wheel_mount.obj scale=1 1 1
Joints:
- removed joint revolute_1_0
- removed joint revolute_2_0
- removed joint revolute_3_0
- added joint wheel_1: type revolute, parent omni_wheel_mount_2, child omni_wheel, origin xyz=-6.93889e-18 -1.38778e-17 0.007175 rpy=0 -1.5708 -1.26789, axis -1 0 0, limit effort=2.94 velocity=4.71
- added joint wheel_2: type revolute, parent omni_wheel_mount, child omni_wheel_1, origin xyz=2.77556e-17 -6.93889e-18 0.007175 rpy=0 -1.5708 4.3619, axis -1 0 0, limit effort=2.94 velocity=4.71
- added joint wheel_3: type revolute, parent omni_wheel_mount_1, child omni_wheel_2, origin xyz=0 -1.2753e-17 0.007175 rpy=0 -1.5708 1.81363, axis -1 0 0, limit effort=2.94 velocity=4.71
- joint fastened_6_0: child omni_wheel_mount_v5_1 -> omni_wheel_mount_1
- joint fastened_7_0: child omni_wheel_mount_v5_2 -> omni_wheel_mount_2
- joint fastened_8_0: child omni_wheel_mount_v5 -> omni_wheel_mount

Commit message: fix: update elrobot kinematic tree (wheels first)

File: src/humanoid/robots/assets/elrobot_mobile/urdf/elrobot_mobile.urdf (robot description, URDF)
Before this commit: robot elrobot_mobile, 31 links, 30 joints
Joints:
- removed joint rev_motor_01
- removed joint rev_motor_02
- removed joint rev_motor_03
- removed joint rev_motor_04
- removed joint rev_motor_05
- removed joint rev_motor_06
- removed joint rev_motor_07
- removed joint rev_motor_08
- removed joint rev_motor_08_1
- removed joint rev_motor_08_2
- added joint arm_1: type revolute, parent ST3215_1_v1_1, child Joint_01_1, origin xyz=0.0 0.034904 0.017505 rpy=0 0 0, axis 0.0 -0.008727 0.999962, limit lower=-1.5509 upper=1.5509 effort=2.94 velocity=4.71
- added joint arm_2: type revolute, parent ST3215_2_v1_1, child Joint_02_1, origin xyz=-0.020293 -0.000308 0.035233 rpy=0 0 0, axis -0.999962 -7.6e-05 0.008726, limit lower=-1.6122 upper=1.6122 effort=2.94 velocity=4.71
- added joint arm_3: type revolute, parent ST3215_3_v1_1, child Joint_03_v1_1, origin xyz=-0.019985 -0.000309 0.035408 rpy=0 0 0, axis -0.999848 -0.000152 0.017452, limit lower=-1.7610 upper=1.7610 effort=2.94 velocity=4.71
- added joint arm_4: type revolute, parent ST3215_4_v1_1, child Joint_04_v1_1, origin xyz=-0.02029 0.035229 0.000662 rpy=0 0 0, axis -0.99981 0.008574 0.017527, limit lower=-1.7533 upper=1.7533 effort=2.94 velocity=4.71
- added joint arm_5: type revolute, parent ST3215_5_v1_1, child Joint_05_v1_1, origin xyz=0.000323 0.0172 0.010051 rpy=0 0 0, axis -0.008573 -0.999963 0.000151, limit lower=-3.1907 upper=2.6998 effort=2.94 velocity=4.71
- added joint arm_6: type revolute, parent ST3215_6_v1_1, child Joint_06_v1_1, origin xyz=-0.019988 0.035407 0.000351 rpy=0 0 0, axis -0.999697 0.0173 0.017525, limit lower=-1.3775 upper=1.7641 effort=2.94 velocity=4.71
- added joint arm_7: type revolute, parent ST3215_7_v1_1, child Gripper_Base_v1_1, origin xyz=0.000473 0.017284 0.009899 rpy=0 0 0, axis -0.017144 -0.999812 0.009029, limit lower=-3.0710 upper=2.7796 effort=2.94 velocity=4.71
- added joint gripper_1: type revolute, parent ST3215_8_v1_1, child Gripper_Gear_v1_1, origin xyz=0.0 0.0 0.0 rpy=0 0 0, axis 0.017144 0.999812 -0.009029, limit lower=0 upper=2.2028 effort=2.94 velocity=4.71
- added joint gripper_2: type prismatic, parent Gripper_Base_v1_1, child Gripper_Jaw_02_v1_1, origin xyz=0.311734 -0.199648 0.032849 rpy=0 0 0, axis -0.999697 0.0173 0.017525, limit lower=-0.0255 upper=0.0 effort=2.94 velocity=4.71, mimic joint=gripper_1 multiplier=-0.0115 offset=0
- added joint gripper_3: type prismatic, parent Gripper_Base_v1_1, child Gripper_Jaw_01_v1_1, origin xyz=0.308573 -0.243367 -0.049391 rpy=0 0 0, axis -0.999697 0.0173 0.017525, limit lower=0.0 upper=0.0255 effort=2.94 velocity=4.71, mimic joint=gripper_1 multiplier=0.0115 offset=0
- joint base_to_arm: origin xyz=-0.091 -0.016 0.007 rpy=0 0 0 -> xyz=0 0.036 0.007 rpy=0 0 0
- joint fastened_5_0: axis 0.5 -0.866025 0 -> 0 0 -1; child base_plate_upper -> omni_wheel_mount_1; origin xyz=-0.0454 6.31089e-30 1.38778e-17 rpy=1.5708 -1.0472 -1.5708 -> xyz=-0.0102 3.22103e-18 0.0042 rpy=-1.2326e-32 -1.88299e-45 -5.43003e-45; parent sts3215_03a_v1_2 -> sts3215_03a_v1
- joint fastened_6_0: axis 0 0 -1 -> 0 0 1; child omni_wheel_mount_1 -> omni_wheel_mount_2; origin xyz=-0.0102 3.22103e-18 0.0042 rpy=-1.2326e-32 -1.88299e-45 -5.43003e-45 -> xyz=-0.0102 6.31089e-30 0.0042 rpy=6.77927e-32 2.18953e-46 1.36846e-47; parent sts3215_03a_v1 -> sts3215_03a_v1_2
- joint fastened_7_0: axis 0 0 1 -> 0 0 -1; child omni_wheel_mount_2 -> omni_wheel_mount; origin xyz=-0.0102 6.31089e-30 0.0042 rpy=6.77927e-32 2.18953e-46 1.36846e-47 -> xyz=-0.0102 6.93889e-18 0.0042 rpy=8.32667e-17 1.35751e-45 1.97058e-46; parent sts3215_03a_v1_2 -> sts3215_03a_v1_1
- joint fastened_8_0: child omni_wheel_mount -> base_plate_upper; origin xyz=-0.0102 6.93889e-18 0.0042 rpy=8.32667e-17 1.35751e-45 1.97058e-46 -> xyz=0 0 0.053 rpy=0 -0 0; parent sts3215_03a_v1_1 -> base_plate_lower
- joint wheel_1: child omni_wheel -> omni_wheel_2; origin xyz=-6.93889e-18 -1.38778e-17 0.007175 rpy=0 -1.5708 -1.26789 -> xyz=0 -7.11514e-18 0.007175 rpy=0 -1.5708 0.279327; parent omni_wheel_mount_2 -> omni_wheel_mount_1; type revolute -> continuous
- joint wheel_2: child omni_wheel_1 -> omni_wheel; origin xyz=2.77556e-17 -6.93889e-18 0.007175 rpy=0 -1.5708 4.3619 -> xyz=-6.93889e-18 -1.38778e-17 0.007175 rpy=0 -1.5708 -1.26789; parent omni_wheel_mount -> omni_wheel_mount_2; type revolute -> continuous
- joint wheel_3: child omni_wheel_2 -> omni_wheel_1; origin xyz=0 -1.2753e-17 0.007175 rpy=0 -1.5708 1.81363 -> xyz=1.04083e-17 -1.38778e-17 0.007175 rpy=0 -1.5708 4.3619; parent omni_wheel_mount_1 -> omni_wheel_mount; type revolute -> continuous

Commit message: feat: add base pose and velocity commands
chore: add elrobot_mobile config

File: src/humanoid/robots/assets/elrobot_mobile/urdf/elrobot_mobile.urdf (robot description, URDF)
Before this commit: robot elrobot_mobile, 31 links, 30 joints
Joints:
- joint wheel_1: limit effort=2.94 velocity=4.71 -> lower=-1e9 upper=1e9 effort=2.94 velocity=4.71; type continuous -> revolute
- joint wheel_2: limit effort=2.94 velocity=4.71 -> lower=-1e9 upper=1e9 effort=2.94 velocity=4.71; type continuous -> revolute
- joint wheel_3: limit effort=2.94 velocity=4.71 -> lower=-1e9 upper=1e9 effort=2.94 velocity=4.71; type continuous -> revolute

Commit message: feat: properly handle generalized position/velocity in RobotState and RobotJointCommand
fix: use continuous joints for elrobot_mobile wheels

File: src/humanoid/robots/assets/elrobot_mobile/urdf/elrobot_mobile.urdf (robot description, URDF)
Before this commit: robot elrobot_mobile, 31 links, 30 joints
Joints:
- joint wheel_1: limit lower=-1e9 upper=1e9 effort=2.94 velocity=4.71 -> effort=2.94 velocity=4.71; type revolute -> continuous
- joint wheel_2: limit lower=-1e9 upper=1e9 effort=2.94 velocity=4.71 -> effort=2.94 velocity=4.71; type revolute -> continuous
- joint wheel_3: limit lower=-1e9 upper=1e9 effort=2.94 velocity=4.71 -> effort=2.94 velocity=4.71; type revolute -> continuous

Commit message: feat: add wheel tasks to OSC + wheel frames to elrobot_mobile URDF + WheelConfig to RobotConfig
fix: transform tool relative to base in Action instead of OSC (correctly publishes commands)

File: src/humanoid/robots/assets/elrobot_mobile/urdf/elrobot_mobile.urdf (robot description, URDF)
Before this commit: robot elrobot_mobile, 31 links, 30 joints
Links:
- added link wheel_1_floor
- added link wheel_2_floor
- added link wheel_3_floor
Joints:
- added joint wheel_1_floor_joint: type fixed, parent root, child wheel_1_floor, origin xyz=0 0 0 rpy=0 0 3.141593
- added joint wheel_2_floor_joint: type fixed, parent root, child wheel_2_floor, origin xyz=0 0 0 rpy=0 0 -1.047198
- added joint wheel_3_floor_joint: type fixed, parent root, child wheel_3_floor, origin xyz=0 0 0 rpy=0 0 1.047198

Commit message: fix: correct mesh names for elrobot_mobile.urdf (+ add default mesh collision geometries)

File: src/humanoid/robots/assets/elrobot_mobile/urdf/elrobot_mobile.urdf (robot description, URDF)
Before this commit: robot elrobot_mobile, 34 links, 33 joints
Links:
- link base_plate_lower: geometry collision mesh filename=package://elrobot_mobile/meshes/base_plate_lower.obj scale=1 1 1; visual mesh filename=package://elrobot_mobile/meshes/base_plate_lower.obj scale=1 1 1
- link base_plate_upper: geometry collision mesh filename=package://elrobot_mobile/meshes/base_plate_upper.obj scale=1 1 1; visual mesh filename=package://elrobot_mobile/meshes/base_plate_upper.obj scale=1 1 1
- link omni_wheel: geometry collision mesh filename=package://elrobot_mobile/meshes/omni_wheel.obj scale=1 1 1; visual mesh filename=package://elrobot_mobile/meshes/omni_wheel.obj scale=1 1 1
- link omni_wheel_1: geometry collision mesh filename=package://elrobot_mobile/meshes/omni_wheel.obj scale=1 1 1; visual mesh filename=package://elrobot_mobile/meshes/omni_wheel.obj scale=1 1 1
- link omni_wheel_2: geometry collision mesh filename=package://elrobot_mobile/meshes/omni_wheel.obj scale=1 1 1; visual mesh filename=package://elrobot_mobile/meshes/omni_wheel.obj scale=1 1 1
- link omni_wheel_mount: geometry collision mesh filename=package://elrobot_mobile/meshes/omni_wheel_mount.obj scale=1 1 1; visual mesh filename=package://elrobot_mobile/meshes/omni_wheel_mount.obj scale=1 1 1
- link omni_wheel_mount_1: geometry collision mesh filename=package://elrobot_mobile/meshes/omni_wheel_mount.obj scale=1 1 1; visual mesh filename=package://elrobot_mobile/meshes/omni_wheel_mount.obj scale=1 1 1
- link omni_wheel_mount_2: geometry collision mesh filename=package://elrobot_mobile/meshes/omni_wheel_mount.obj scale=1 1 1; visual mesh filename=package://elrobot_mobile/meshes/omni_wheel_mount.obj scale=1 1 1
- link sts3215_03a_v1: geometry collision mesh filename=package://elrobot_mobile/meshes/STS3215_03a_v1.obj scale=1 1 1; visual mesh filename=package://elrobot_mobile/meshes/STS3215_03a_v1.obj scale=1 1 1
- link sts3215_03a_v1_1: geometry collision mesh filename=package://elrobot_mobile/meshes/STS3215_03a_v1.obj scale=1 1 1; visual mesh filename=package://elrobot_mobile/meshes/STS3215_03a_v1.obj scale=1 1 1
- link sts3215_03a_v1_2: geometry collision mesh filename=package://elrobot_mobile/meshes/STS3215_03a_v1.obj scale=1 1 1; visual mesh filename=package://elrobot_mobile/meshes/STS3215_03a_v1.obj scale=1 1 1

Commit message: fix: revert lower-case omni_wheel.obj naming due to .MTL reference

File: src/humanoid/robots/assets/elrobot_mobile/urdf/elrobot_mobile.urdf (robot description, URDF)
Before this commit: robot elrobot_mobile, 34 links, 33 joints
Links:
- link omni_wheel: geometry collision mesh filename=package://elrobot_mobile/meshes/Omni_Wheel.obj scale=1 1 1; visual mesh filename=package://elrobot_mobile/meshes/Omni_Wheel.obj scale=1 1 1
- link omni_wheel_1: geometry collision mesh filename=package://elrobot_mobile/meshes/Omni_Wheel.obj scale=1 1 1; visual mesh filename=package://elrobot_mobile/meshes/Omni_Wheel.obj scale=1 1 1
- link omni_wheel_2: geometry collision mesh filename=package://elrobot_mobile/meshes/Omni_Wheel.obj scale=1 1 1; visual mesh filename=package://elrobot_mobile/meshes/Omni_Wheel.obj scale=1 1 1

File: src/humanoid/robots/assets/elrobot_mobile/urdf/elrobot_mobile_collision.urdf (robot description, URDF)
Before this commit: robot elrobot_mobile, 34 links, 33 joints
Links:
- link omni_wheel: geometry collision sphere radius=0.055; visual mesh filename=package://elrobot_mobile/meshes/Omni_Wheel.obj scale=1 1 1
- link omni_wheel_1: geometry collision sphere radius=0.055; visual mesh filename=package://elrobot_mobile/meshes/Omni_Wheel.obj scale=1 1 1
- link omni_wheel_2: geometry visual mesh filename=package://elrobot_mobile/meshes/Omni_Wheel.obj scale=1 1 1
