Commit message: refactor(robots): simplify URDF asset naming
- replace generated joint, link, and mesh names with semantic names
- flatten SO-101 meshes and consolidate mobile OBJ materials
- validate URDF, SRDF, and mesh references

File: src/humanoid/robots/assets/elrobot_mobile/urdf/elrobot_mobile_collision.urdf (robot description, URDF)
Before this commit: robot elrobot_mobile, 34 links, 33 joints
Links:
- removed link Gripper_Base_v1_1
- removed link Gripper_Gear_v1_1
- removed link Gripper_Jaw_01_v1_1
- removed link Gripper_Jaw_02_v1_1
- removed link Joint_01_1
- removed link Joint_02_1
- removed link Joint_03_v1_1
- removed link Joint_04_v1_1
- removed link Joint_05_v1_1
- removed link Joint_06_v1_1
- removed link ST3215_1_v1_1
- removed link ST3215_2_v1_1
- removed link ST3215_3_v1_1
- removed link ST3215_4_v1_1
- removed link ST3215_5_v1_1
- removed link ST3215_6_v1_1
- removed link ST3215_7_v1_1
- removed link ST3215_8_v1_1
- removed link base_plate_lower
- removed link base_plate_upper
- removed link omni_wheel
- removed link omni_wheel_1
- removed link omni_wheel_2
- removed link omni_wheel_mount
- removed link omni_wheel_mount_1
- removed link omni_wheel_mount_2
- removed link root
- removed link sts3215_03a_v1
- removed link sts3215_03a_v1_1
- removed link sts3215_03a_v1_2
- added link arm_1_link, mass 0.05706; collision cylinder length=0.058917 radius=0.028189; collision sphere radius=0.028189
- added link arm_2_link, mass 0.05084; collision cylinder length=0.0783 radius=0.031753; collision sphere radius=0.031753
- added link arm_3_link, mass 0.03822; visual mesh filename=package://elrobot/meshes/arm_3.stl scale=0.001 0.001 0.001
- added link arm_4_link, mass 0.05152; collision cylinder length=0.089987 radius=0.034461; collision sphere radius=0.034461
- added link arm_5_link, mass 0.01756; visual mesh filename=package://elrobot/meshes/arm_5.stl scale=0.001 0.001 0.001
- added link arm_6_link, mass 0.03882; collision cylinder length=0.06323 radius=0.034461; collision sphere radius=0.034461
- added link arm_base_link, mass 0.03944; collision cylinder length=0.12 radius=0.045243; collision sphere radius=0.045243
- added link finger_1_link, mass 0.0125; visual mesh filename=package://elrobot/meshes/finger_1.stl scale=0.001 0.001 0.001
- added link finger_2_link, mass 0.0125; visual mesh filename=package://elrobot/meshes/finger_2.stl scale=0.001 0.001 0.001
- added link finger_drive_link, mass 0.055; collision sphere radius=0.03; visual mesh filename=package://elrobot/meshes/servo_8.stl scale=0.001 0.001 0.001
- added link gripper_base_link, mass 0.06244; collision cylinder length=0.05 radius=0.05; collision sphere radius=0.05
- added link gripper_gear_link, mass 0.0039; visual mesh filename=package://elrobot/meshes/gripper_gear.stl scale=0.001 0.001 0.001
- added link lower_plate_link, mass 0.000248008; visual mesh filename=package://elrobot_mobile/meshes/lower_plate.obj scale=1 1 1
- added link motor_1_link, mass 0.055; visual mesh filename=package://elrobot/meshes/servo_1.stl scale=0.001 0.001 0.001
- added link motor_2_link, mass 0.055; visual mesh filename=package://elrobot/meshes/servo_2.stl scale=0.001 0.001 0.001
- added link motor_3_link, mass 0.055; visual mesh filename=package://elrobot/meshes/servo_3.stl scale=0.001 0.001 0.001
- added link motor_4_link, mass 0.055; visual mesh filename=package://elrobot/meshes/servo_4.stl scale=0.001 0.001 0.001
- added link motor_5_link, mass 0.055; visual mesh filename=package://elrobot/meshes/servo_5.stl scale=0.001 0.001 0.001
- added link motor_6_link, mass 0.055; visual mesh filename=package://elrobot/meshes/servo_6.stl scale=0.001 0.001 0.001
- added link motor_7_link, mass 0.055; visual mesh filename=package://elrobot/meshes/servo_7.stl scale=0.001 0.001 0.001
- added link upper_plate_link, mass 0.000242412; visual mesh filename=package://elrobot_mobile/meshes/upper_plate.obj scale=1 1 1
- added link wheel_1_link, mass 0.000188807; visual mesh filename=package://elrobot_mobile/meshes/wheel.obj scale=1 1 1
- added link wheel_1_motor_link, mass 3.6217e-05; visual mesh filename=package://elrobot_mobile/meshes/servo.obj scale=1 1 1
- added link wheel_1_mount_link, mass 1.57415e-05; visual mesh filename=package://elrobot_mobile/meshes/wheel_mount.obj scale=1 1 1
- added link wheel_2_link, mass 0.000188807; collision sphere radius=0.055; visual mesh filename=package://elrobot_mobile/meshes/wheel.obj scale=1 1 1
- added link wheel_2_motor_link, mass 3.6217e-05; visual mesh filename=package://elrobot_mobile/meshes/servo.obj scale=1 1 1
- added link wheel_2_mount_link, mass 1.57415e-05; visual mesh filename=package://elrobot_mobile/meshes/wheel_mount.obj scale=1 1 1
- added link wheel_3_link, mass 0.000188807; collision sphere radius=0.055; visual mesh filename=package://elrobot_mobile/meshes/wheel.obj scale=1 1 1
- added link wheel_3_motor_link, mass 3.6217e-05; visual mesh filename=package://elrobot_mobile/meshes/servo.obj scale=1 1 1
- added link wheel_3_mount_link, mass 1.57415e-05; visual mesh filename=package://elrobot_mobile/meshes/wheel_mount.obj scale=1 1 1
- link base_link: mass 0.03944 -> None; geometry 
Joints:
- removed joint Rigid 1
- removed joint Rigid 11
- removed joint Rigid 13
- removed joint Rigid 15
- removed joint Rigid 17
- removed joint Rigid 3
- removed joint Rigid 7
- removed joint Rigid 9
- removed joint base_to_arm
- removed joint fastened_1_0
- removed joint fastened_2_0
- removed joint fastened_3_0
- removed joint fastened_4_0
- removed joint fastened_5_0
- removed joint fastened_6_0
- removed joint fastened_7_0
- removed joint fastened_8_0
- added joint arm_mount: type fixed, parent upper_plate_link, child arm_base_link, origin xyz=0 0.036 0.007 rpy=0 0 0
- added joint base_mount: type fixed, parent base_link, child lower_plate_link, origin xyz=0 0 -8.67362e-19 rpy=0 -0 0, axis 0 0 -1
- added joint finger_drive_mount: type fixed, parent gripper_base_link, child finger_drive_link, origin xyz=0.000776 0.045242 -0.000409 rpy=0 0 0
- added joint motor_1_mount: type fixed, parent arm_base_link, child motor_1_link, origin xyz=0.0 0.007585 0.0315 rpy=0 0 0
- added joint motor_2_mount: type fixed, parent arm_1_link, child motor_2_link, origin xyz=0.000625 -5.8e-05 0.0067 rpy=0 0 0
- added joint motor_3_mount: type fixed, parent arm_2_link, child motor_3_link, origin xyz=0.019863 -0.000487 0.055827 rpy=0 0 0
- added joint motor_4_mount: type fixed, parent arm_3_link, child motor_4_link, origin xyz=0.021263 0.001933 0.036403 rpy=0 0 0
- added joint motor_5_mount: type fixed, parent arm_4_link, child motor_5_link, origin xyz=0.020391 0.065663 -0.010035 rpy=0 0 0
- added joint motor_6_mount: type fixed, parent arm_5_link, child motor_6_link, origin xyz=6.5e-05 0.0075 -1e-06 rpy=0 0 0
- added joint motor_7_mount: type fixed, parent arm_6_link, child motor_7_link, origin xyz=0.020478 0.038023 -0.010611 rpy=0 0 0
- added joint wheel_1_bracket_mount: type fixed, parent wheel_1_motor_link, child wheel_1_mount_link, origin xyz=-0.0102 3.22103e-18 0.0042 rpy=-1.2326e-32 -1.88299e-45 -5.43003e-45, axis 0 0 -1
- added joint wheel_1_motor_mount: type fixed, parent lower_plate_link, child wheel_1_motor_link, origin xyz=1.94313e-14 -0.105 0.007 rpy=0 1.5708 4.71239, axis 0 1 0
- added joint wheel_2_bracket_mount: type fixed, parent wheel_2_motor_link, child wheel_2_mount_link, origin xyz=-0.0102 6.31089e-30 0.0042 rpy=6.77927e-32 2.18953e-46 1.36846e-47, axis 0 0 1
- added joint wheel_2_motor_mount: type fixed, parent lower_plate_link, child wheel_2_motor_link, origin xyz=0.0909327 0.0525 0.007 rpy=0 1.5708 0.523599, axis 0 1 0
- added joint wheel_3_bracket_mount: type fixed, parent wheel_3_motor_link, child wheel_3_mount_link, origin xyz=-0.0102 6.93889e-18 0.0042 rpy=8.32667e-17 1.35751e-45 1.97058e-46, axis 0 0 -1
- added joint wheel_3_motor_mount: type fixed, parent lower_plate_link, child wheel_3_motor_link, origin xyz=-0.0909327 0.0525 0.007 rpy=0 1.5708 2.61799, axis 0 1 0
- added joint wheel_platform_mount: type fixed, parent lower_plate_link, child upper_plate_link, origin xyz=0 0 0.053 rpy=0 -0 0, axis 0 0 -1
- joint arm_1: child Joint_01_1 -> arm_1_link; parent ST3215_1_v1_1 -> motor_1_link
- joint arm_2: child Joint_02_1 -> arm_2_link; parent ST3215_2_v1_1 -> motor_2_link
- joint arm_3: child Joint_03_v1_1 -> arm_3_link; parent ST3215_3_v1_1 -> motor_3_link
- joint arm_4: child Joint_04_v1_1 -> arm_4_link; parent ST3215_4_v1_1 -> motor_4_link
- joint arm_5: child Joint_05_v1_1 -> arm_5_link; parent ST3215_5_v1_1 -> motor_5_link
- joint arm_6: child Joint_06_v1_1 -> arm_6_link; parent ST3215_6_v1_1 -> motor_6_link
- joint arm_7: child Gripper_Base_v1_1 -> gripper_base_link; parent ST3215_7_v1_1 -> motor_7_link
- joint gripper_1: child Gripper_Gear_v1_1 -> gripper_gear_link; parent ST3215_8_v1_1 -> finger_drive_link
- joint gripper_2: child Gripper_Jaw_02_v1_1 -> finger_2_link; parent Gripper_Base_v1_1 -> gripper_base_link
- joint gripper_3: child Gripper_Jaw_01_v1_1 -> finger_1_link; parent Gripper_Base_v1_1 -> gripper_base_link
- joint wheel_1: child omni_wheel_2 -> wheel_1_link; parent omni_wheel_mount_1 -> wheel_1_mount_link
- joint wheel_1_floor_joint: parent root -> base_link
- joint wheel_2: child omni_wheel -> wheel_2_link; parent omni_wheel_mount_2 -> wheel_2_mount_link
- joint wheel_2_floor_joint: parent root -> base_link
- joint wheel_3: child omni_wheel_1 -> wheel_3_link; parent omni_wheel_mount -> wheel_3_mount_link
- joint wheel_3_floor_joint: parent root -> base_link

File: src/humanoid/robots/assets/so101/urdf/so101.urdf (robot description, URDF)
Before this commit: robot so101_new_calib, 8 links, 7 joints
Links:
- removed link gripper_frame_link
- removed link moving_jaw_so101_v1_link
- added link moving_jaw_link, mass 0.012; collision mesh filename=package://so101/meshes/moving_jaw.stl; visual mesh filename=package://so101/meshes/moving_jaw.stl
- added link tool_link, mass 1e-9
- link base_link: geometry collision mesh filename=package://so101/meshes/base.stl; collision mesh filename=package://so101/meshes/base_motor_mount.stl
- link gripper_link: geometry collision mesh filename=package://so101/meshes/gripper_mount.stl; collision mesh filename=package://so101/meshes/servo.stl
- link lower_arm_link: geometry collision mesh filename=package://so101/meshes/lower_arm.stl; collision mesh filename=package://so101/meshes/servo.stl
- link shoulder_link: geometry collision mesh filename=package://so101/meshes/servo.stl; collision mesh filename=package://so101/meshes/shoulder_bracket.stl
- link upper_arm_link: geometry collision mesh filename=package://so101/meshes/servo.stl; collision mesh filename=package://so101/meshes/upper_arm.stl
- link wrist_link: geometry collision mesh filename=package://so101/meshes/servo_no_horn.stl; collision mesh filename=package://so101/meshes/wrist_bracket.stl
Joints:
- removed joint gripper_frame_joint
- added joint tool_joint: type fixed, parent gripper_link, child tool_link, origin xyz=-0.0079 -0.000218121 -0.0981274 rpy=0 3.14159 0, axis 0 0 0
- joint gripper: child moving_jaw_so101_v1_link -> moving_jaw_link
