Commit message: feat: add onboard robot operation workflows
Start and reconnect the Meta Quest bridge with persistent ADB authorization. Persist recordings, add Raspberry Pi dashboard and sync helpers, adjust the model and dashboard mark, and expand runtime coverage.

File: ros_ws/src/triskel_description/urdf/triskel.urdf (robot description, URDF)
Before this commit: robot triskel, 34 links, 33 joints
Joints:
- joint base_mount: origin xyz=0 0 -8.67362e-19 rpy=0 -0 0 -> xyz=0 0 0.0321 rpy=0 -0 0

Commit message: fix(hardware): align robot coordinates with STS feedback
- reverse arm axes and asymmetric limits for the STS sign convention
- transform Home and Rest coordinates while preserving physical poses
- restore the gripper range to [-2.2, 0]
- define Home as gripper-open and Rest as gripper-closed
- drive gripper teleop toward named endpoints
- update keyboard, Meta Quest, homing, and regression tests

File: ros_ws/src/triskel_description/urdf/triskel.urdf (robot description, URDF)
Before this commit: robot triskel, 34 links, 33 joints
Joints:
- joint arm_1: axis 0.0 -0.008727 0.999962 -> 0.0 0.008727 -0.999962
- joint arm_2: axis -0.999962 -7.6e-05 0.008726 -> 0.999962 7.6e-05 -0.008726
- joint arm_3: axis -0.999848 -0.000152 0.017452 -> 0.999848 0.000152 -0.017452
- joint arm_4: axis -0.99981 0.008574 0.017527 -> 0.99981 -0.008574 -0.017527
- joint arm_5: axis -0.008573 -0.999963 0.000151 -> 0.008573 0.999963 -0.000151; limit lower=-3.1907 upper=2.6998 effort=2.94 velocity=4.71 -> lower=-2.6998 upper=3.1907 effort=2.94 velocity=4.71
- joint arm_6: axis -0.999697 0.0173 0.017525 -> 0.999697 -0.0173 -0.017525; limit lower=-1.3775 upper=1.7641 effort=2.94 velocity=4.71 -> lower=-1.7641 upper=1.3775 effort=2.94 velocity=4.71
- joint arm_7: axis -0.017144 -0.999812 0.009029 -> 0.017144 0.999812 -0.009029; limit lower=-3.0710 upper=2.7796 effort=2.94 velocity=4.71 -> lower=-2.7796 upper=3.0710 effort=2.94 velocity=4.71

File: ros_ws/src/triskel_hardware/urdf/triskel.ros2_control.xacro (robot description, xacro)
@@ -65,7 +65,7 @@
       <xacro:position_joint name="arm_3" motor_id="3" lower="-1.7610" upper="1.7610" />
       <xacro:position_joint name="arm_4" motor_id="4" lower="-1.7533" upper="1.7533" />
-      <xacro:position_joint name="arm_5" motor_id="5" lower="-3.1907" upper="2.6998" />
-      <xacro:position_joint name="arm_6" motor_id="6" lower="-1.3775" upper="1.7641" />
-      <xacro:position_joint name="arm_7" motor_id="7" lower="-3.0710" upper="2.7796" />
+      <xacro:position_joint name="arm_5" motor_id="5" lower="-2.6998" upper="3.1907" />
+      <xacro:position_joint name="arm_6" motor_id="6" lower="-1.7641" upper="1.3775" />
+      <xacro:position_joint name="arm_7" motor_id="7" lower="-2.7796" upper="3.0710" />
       <xacro:position_joint
         name="gripper_1"

Commit message: fix(hardware): synchronize startup state and gripper visualization
- seed trajectory controllers from measured joint feedback
- prevent stale command history from triggering false limit enforcement
- align gripper mimic joints with the hardware open/closed convention
- add regression coverage for controller initialization and gripper travel

File: ros_ws/src/triskel_description/urdf/triskel.urdf (robot description, URDF)
Before this commit: robot triskel, 34 links, 33 joints
Joints:
- joint gripper_2: mimic joint=gripper_1 multiplier=0.0115 offset=0 -> joint=gripper_1 multiplier=-0.0115 offset=-0.0253
- joint gripper_3: mimic joint=gripper_1 multiplier=-0.0115 offset=0 -> joint=gripper_1 multiplier=0.0115 offset=0.0253

Commit message: Fix ROS 2 hardware homing and runtime startup

File: ros_ws/src/triskel_description/urdf/triskel.urdf (robot description, URDF)
Before this commit: robot triskel, 34 links, 33 joints
Joints:
- joint arm_5: limit lower=-2.6998 upper=3.1907 effort=2.94 velocity=4.71 -> lower=-2.6998 upper=3.141592653589793 effort=2.94 velocity=4.71
- joint gripper_2: mimic joint=gripper_1 multiplier=-0.0115 offset=-0.0253 -> joint=gripper_1 multiplier=0.0115 offset=0
- joint gripper_3: mimic joint=gripper_1 multiplier=0.0115 offset=0.0253 -> joint=gripper_1 multiplier=-0.0115 offset=0

File: ros_ws/src/triskel_hardware/urdf/triskel.ros2_control.xacro (robot description, xacro)
@@ -7,16 +7,15 @@
     <ros2_control name="triskel_system" type="system">
       <hardware>
-        <xacro:if value="${use_mock_hardware}">
-          <plugin>mock_components/GenericSystem</plugin>
-          <param name="calculate_dynamics">true</param>
-        </xacro:if>
-        <xacro:unless value="${use_mock_hardware}">
-          <plugin>sts_hardware_interface/STSHardwareInterface</plugin>
-          <param name="serial_port">${serial_port}</param>
-          <param name="baud_rate">${baud_rate}</param>
-          <param name="use_sync_write">true</param>
-          <param name="proportional_acc_max">100</param>
-          <param name="reset_states_on_activate">false</param>
-        </xacro:unless>
+        <plugin>sts_hardware_interface/STSHardwareInterface</plugin>
+        <param name="serial_port">${serial_port}</param>
+        <param name="baud_rate">${baud_rate}</param>
+        <param name="communication_timeout_ms">100</param>
+        <param name="use_sync_write">true</param>
+        <param name="enable_mock_mode">${str(use_mock_hardware).lower()}</param>
+        <param name="proportional_acc_max">100</param>
+        <!-- Mode-0 speed is an unsigned cap; direction comes from position. -->
+        <param name="proportional_vel_max">1000</param>
+        <param name="proportional_vel_deadband">0.0</param>
+        <param name="reset_states_on_activate">false</param>
       </hardware>
       <xacro:macro name="velocity_joint" params="name motor_id">
@@ -25,4 +24,5 @@
           <param name="operating_mode">1</param>
           <param name="max_velocity_steps">3400</param>
+          <param name="max_velocity">4.71</param>
           <command_interface name="velocity">
             <param name="min">-4.71</param>
@@ -34,4 +34,8 @@
           <state_interface name="velocity" />
           <state_interface name="effort" />
+          <state_interface name="voltage" />
+          <state_interface name="temperature" />
+          <state_interface name="current" />
+          <state_interface name="is_moving" />
         </joint>
       </xacro:macro>
@@ -47,8 +51,10 @@
           <param name="max_position">${upper}</param>
           <param name="max_velocity_steps">3400</param>
+          <param name="max_velocity">4.71</param>
           <command_interface name="position">
             <param name="min">${lower}</param>
             <param name="max">${upper}</param>
           </command_interface>
+          <!-- Mode 0 uses position only; the driver supplies its speed cap. -->
           <state_interface name="position">
             <param name="initial_value">0.0</param>
@@ -56,4 +62,8 @@
           <state_interface name="velocity" />
           <state_interface name="effort" />
+          <state_interface name="voltage" />
+          <state_interface name="temperature" />
+          <state_interface name="current" />
+          <state_interface name="is_moving" />
         </joint>
       </xacro:macro>
@@ -65,5 +75,5 @@
       <xacro:position_joint name="arm_3" motor_id="3" lower="-1.7610" upper="1.7610" />
       <xacro:position_joint name="arm_4" motor_id="4" lower="-1.7533" upper="1.7533" />
-      <xacro:position_joint name="arm_5" motor_id="5" lower="-2.6998" upper="3.1907" />
+      <xacro:position_joint name="arm_5" motor_id="5" lower="-2.6998" upper="3.141592653589793" />
       <xacro:position_joint name="arm_6" motor_id="6" lower="-1.7641" upper="1.3775" />
       <xacro:position_joint name="arm_7" motor_id="7" lower="-2.7796" upper="3.0710" />
