Commit message: refactor: rename mobile robot to Triskel
Consolidate the mobile base and arm assets under the Triskel identity, remove the standalone Elrobot configuration, and explicitly stop owned MeshCat servers during visualizer teardown.

File: src/humanoid/robots/assets/triskel/urdf/triskel.urdf (robot description, URDF)
Before this commit: robot elrobot_mobile, 34 links, 33 joints
Links:
- link arm_1_link: geometry collision mesh filename=package://triskel/meshes/arm_1.stl scale=0.001 0.001 0.001; visual mesh filename=package://triskel/meshes/arm_1.stl scale=0.001 0.001 0.001
- link arm_2_link: geometry collision mesh filename=package://triskel/meshes/arm_2.stl scale=0.001 0.001 0.001; visual mesh filename=package://triskel/meshes/arm_2.stl scale=0.001 0.001 0.001
- link arm_3_link: geometry collision mesh filename=package://triskel/meshes/arm_3.stl scale=0.001 0.001 0.001; visual mesh filename=package://triskel/meshes/arm_3.stl scale=0.001 0.001 0.001
- link arm_4_link: geometry collision mesh filename=package://triskel/meshes/arm_4.stl scale=0.001 0.001 0.001; visual mesh filename=package://triskel/meshes/arm_4.stl scale=0.001 0.001 0.001
- link arm_5_link: geometry collision mesh filename=package://triskel/meshes/arm_5.stl scale=0.001 0.001 0.001; visual mesh filename=package://triskel/meshes/arm_5.stl scale=0.001 0.001 0.001
- link arm_6_link: geometry collision mesh filename=package://triskel/meshes/arm_6.stl scale=0.001 0.001 0.001; visual mesh filename=package://triskel/meshes/arm_6.stl scale=0.001 0.001 0.001
- link arm_base_link: geometry collision mesh filename=package://triskel/meshes/base.stl scale=0.001 0.001 0.001; visual mesh filename=package://triskel/meshes/base.stl scale=0.001 0.001 0.001
- link finger_1_link: geometry collision mesh filename=package://triskel/meshes/finger_1.stl scale=0.001 0.001 0.001; visual mesh filename=package://triskel/meshes/finger_1.stl scale=0.001 0.001 0.001
- link finger_2_link: geometry collision mesh filename=package://triskel/meshes/finger_2.stl scale=0.001 0.001 0.001; visual mesh filename=package://triskel/meshes/finger_2.stl scale=0.001 0.001 0.001
- link finger_drive_link: geometry collision mesh filename=package://triskel/meshes/servo_8.stl scale=0.001 0.001 0.001; visual mesh filename=package://triskel/meshes/servo_8.stl scale=0.001 0.001 0.001
- link gripper_base_link: geometry collision mesh filename=package://triskel/meshes/gripper_base.stl scale=0.001 0.001 0.001; visual mesh filename=package://triskel/meshes/gripper_base.stl scale=0.001 0.001 0.001
- link gripper_gear_link: geometry collision mesh filename=package://triskel/meshes/gripper_gear.stl scale=0.001 0.001 0.001; visual mesh filename=package://triskel/meshes/gripper_gear.stl scale=0.001 0.001 0.001
- link lower_plate_link: geometry collision mesh filename=package://triskel/meshes/lower_plate.obj scale=1 1 1; visual mesh filename=package://triskel/meshes/lower_plate.obj scale=1 1 1
- link motor_1_link: geometry collision mesh filename=package://triskel/meshes/servo_1.stl scale=0.001 0.001 0.001; visual mesh filename=package://triskel/meshes/servo_1.stl scale=0.001 0.001 0.001
- link motor_2_link: geometry collision mesh filename=package://triskel/meshes/servo_2.stl scale=0.001 0.001 0.001; visual mesh filename=package://triskel/meshes/servo_2.stl scale=0.001 0.001 0.001
- link motor_3_link: geometry collision mesh filename=package://triskel/meshes/servo_3.stl scale=0.001 0.001 0.001; visual mesh filename=package://triskel/meshes/servo_3.stl scale=0.001 0.001 0.001
- link motor_4_link: geometry collision mesh filename=package://triskel/meshes/servo_4.stl scale=0.001 0.001 0.001; visual mesh filename=package://triskel/meshes/servo_4.stl scale=0.001 0.001 0.001
- link motor_5_link: geometry collision mesh filename=package://triskel/meshes/servo_5.stl scale=0.001 0.001 0.001; visual mesh filename=package://triskel/meshes/servo_5.stl scale=0.001 0.001 0.001
- link motor_6_link: geometry collision mesh filename=package://triskel/meshes/servo_6.stl scale=0.001 0.001 0.001; visual mesh filename=package://triskel/meshes/servo_6.stl scale=0.001 0.001 0.001
- link motor_7_link: geometry collision mesh filename=package://triskel/meshes/servo_7.stl scale=0.001 0.001 0.001; visual mesh filename=package://triskel/meshes/servo_7.stl scale=0.001 0.001 0.001
- link upper_plate_link: geometry collision mesh filename=package://triskel/meshes/upper_plate.obj scale=1 1 1; visual mesh filename=package://triskel/meshes/upper_plate.obj scale=1 1 1
- link wheel_1_link: geometry collision mesh filename=package://triskel/meshes/wheel.obj scale=1 1 1; visual mesh filename=package://triskel/meshes/wheel.obj scale=1 1 1
- link wheel_1_motor_link: geometry collision mesh filename=package://triskel/meshes/servo.obj scale=1 1 1; visual mesh filename=package://triskel/meshes/servo.obj scale=1 1 1
- link wheel_1_mount_link: geometry collision mesh filename=package://triskel/meshes/wheel_mount.obj scale=1 1 1; visual mesh filename=package://triskel/meshes/wheel_mount.obj scale=1 1 1
- link wheel_2_link: geometry collision mesh filename=package://triskel/meshes/wheel.obj scale=1 1 1; visual mesh filename=package://triskel/meshes/wheel.obj scale=1 1 1
- link wheel_2_motor_link: geometry collision mesh filename=package://triskel/meshes/servo.obj scale=1 1 1; visual mesh filename=package://triskel/meshes/servo.obj scale=1 1 1
- link wheel_2_mount_link: geometry collision mesh filename=package://triskel/meshes/wheel_mount.obj scale=1 1 1; visual mesh filename=package://triskel/meshes/wheel_mount.obj scale=1 1 1
- link wheel_3_link: geometry collision mesh filename=package://triskel/meshes/wheel.obj scale=1 1 1; visual mesh filename=package://triskel/meshes/wheel.obj scale=1 1 1
- link wheel_3_motor_link: geometry collision mesh filename=package://triskel/meshes/servo.obj scale=1 1 1; visual mesh filename=package://triskel/meshes/servo.obj scale=1 1 1
- link wheel_3_mount_link: geometry collision mesh filename=package://triskel/meshes/wheel_mount.obj scale=1 1 1; visual mesh filename=package://triskel/meshes/wheel_mount.obj scale=1 1 1

File: src/humanoid/robots/assets/triskel/urdf/triskel_collision.urdf (robot description, URDF)
Before this commit: robot elrobot_mobile, 34 links, 33 joints
Links:
- link arm_1_link: geometry collision cylinder length=0.058917 radius=0.028189; collision sphere radius=0.028189
- link arm_2_link: geometry collision cylinder length=0.0783 radius=0.031753; collision sphere radius=0.031753
- link arm_3_link: geometry visual mesh filename=package://triskel/meshes/arm_3.stl scale=0.001 0.001 0.001
- link arm_4_link: geometry collision cylinder length=0.089987 radius=0.034461; collision sphere radius=0.034461
- link arm_5_link: geometry visual mesh filename=package://triskel/meshes/arm_5.stl scale=0.001 0.001 0.001
- link arm_6_link: geometry collision cylinder length=0.06323 radius=0.034461; collision sphere radius=0.034461
- link arm_base_link: geometry collision cylinder length=0.12 radius=0.045243; collision sphere radius=0.045243
- link finger_1_link: geometry visual mesh filename=package://triskel/meshes/finger_1.stl scale=0.001 0.001 0.001
- link finger_2_link: geometry visual mesh filename=package://triskel/meshes/finger_2.stl scale=0.001 0.001 0.001
- link finger_drive_link: geometry collision sphere radius=0.03; visual mesh filename=package://triskel/meshes/servo_8.stl scale=0.001 0.001 0.001
- link gripper_base_link: geometry collision cylinder length=0.05 radius=0.05; collision sphere radius=0.05
- link gripper_gear_link: geometry visual mesh filename=package://triskel/meshes/gripper_gear.stl scale=0.001 0.001 0.001
- link lower_plate_link: geometry visual mesh filename=package://triskel/meshes/lower_plate.obj scale=1 1 1
- link motor_1_link: geometry visual mesh filename=package://triskel/meshes/servo_1.stl scale=0.001 0.001 0.001
- link motor_2_link: geometry visual mesh filename=package://triskel/meshes/servo_2.stl scale=0.001 0.001 0.001
- link motor_3_link: geometry visual mesh filename=package://triskel/meshes/servo_3.stl scale=0.001 0.001 0.001
- link motor_4_link: geometry visual mesh filename=package://triskel/meshes/servo_4.stl scale=0.001 0.001 0.001
- link motor_5_link: geometry visual mesh filename=package://triskel/meshes/servo_5.stl scale=0.001 0.001 0.001
- link motor_6_link: geometry visual mesh filename=package://triskel/meshes/servo_6.stl scale=0.001 0.001 0.001
- link motor_7_link: geometry visual mesh filename=package://triskel/meshes/servo_7.stl scale=0.001 0.001 0.001
- link upper_plate_link: geometry visual mesh filename=package://triskel/meshes/upper_plate.obj scale=1 1 1
- link wheel_1_link: geometry visual mesh filename=package://triskel/meshes/wheel.obj scale=1 1 1
- link wheel_1_motor_link: geometry visual mesh filename=package://triskel/meshes/servo.obj scale=1 1 1
- link wheel_1_mount_link: geometry visual mesh filename=package://triskel/meshes/wheel_mount.obj scale=1 1 1
- link wheel_2_link: geometry collision sphere radius=0.055; visual mesh filename=package://triskel/meshes/wheel.obj scale=1 1 1
- link wheel_2_motor_link: geometry visual mesh filename=package://triskel/meshes/servo.obj scale=1 1 1
- link wheel_2_mount_link: geometry visual mesh filename=package://triskel/meshes/wheel_mount.obj scale=1 1 1
- link wheel_3_link: geometry collision sphere radius=0.055; visual mesh filename=package://triskel/meshes/wheel.obj scale=1 1 1
- link wheel_3_motor_link: geometry visual mesh filename=package://triskel/meshes/servo.obj scale=1 1 1
- link wheel_3_mount_link: geometry visual mesh filename=package://triskel/meshes/wheel_mount.obj scale=1 1 1
